Commit message: Configurable control methods and gazebo GUI

File: qutms_sim/urdf/gz_plugins.urdf.xacro (robot description, xacro)
@@ -20,34 +20,45 @@
   -->
   <xacro:arg name="namespace" default="sim"/>
-  <!-- Vehicle Dynamics Plugin - DISABLED for ROS 2 Control Testing -->
   <!--
-    IMPORTANT: This plugin uses WorldPoseCmd for kinematic control, which conflicts
-    with physics-based ROS 2 Control. Uncomment this to use custom vehicle control.
-  <gazebo>
-    <plugin filename="libgazebo_vehicle.so" name="gazebo_plugins::vehicle_plugins::VehiclePlugin">
-      <ros>
-        <namespace>/$(arg namespace)</namespace>
-      </ros>
-      <vehicle_params>$(find qutms_sim)/config/vehicle_params.yaml</vehicle_params>
-      <update_rate>50.0</update_rate>
-      <steering_lock_time>1.5</steering_lock_time>
-    </plugin>
-  </gazebo>
+    Control backend selection.
+    control_mode == "dynamic_model" -> custom kinematic vehicle dynamics + control plugins (below)
+    control_mode == "ros2_control"  -> gz_ros2_control physics-based control (at bottom of file)
+    Set via the `control_mode` param in config/global_config.yaml.
   -->
-  <!-- Vehicle Control Plugin - DISABLED (requires vehicle dynamics plugin) -->
-  <!--
-  <gazebo>
-    <plugin filename="libgazebo_vehicle_control.so" name="gazebo_plugins::vehicle_plugins::VehicleControlPlugin">
-      <ros>
-        <namespace>/$(arg namespace)</namespace>
-      </ros>
-      <control_delay>0.035</control_delay>
-      <enable_ackermann>true</enable_ackermann>
-      <enable_twist>true</enable_twist>
-      <ackermann_topic>control/ackermann_cmd</ackermann_topic>
-      <twist_topic>control/twist_cmd</twist_topic>
-    </plugin>
-  </gazebo>
-  -->
+  <xacro:arg name="control_mode" default="dynamic_model"/>
+  <xacro:property name="control_mode" value="$(arg control_mode)"/>
+  <!-- ============================================================= -->
+  <!-- DYNAMIC MODEL BACKEND (kinematic vehicle dynamics)            -->
+  <!-- ============================================================= -->
+  <xacro:if value="${control_mode == 'dynamic_model'}">
+    <!-- Vehicle Dynamics Plugin -->
+    <!--
+      IMPORTANT: This plugin uses WorldPoseCmd for kinematic control, which conflicts
+      with physics-based ROS 2 Control. Only active when control_mode == "dynamic_model".
+    -->
+    <gazebo>
+      <plugin filename="libgazebo_vehicle.so" name="gazebo_plugins::vehicle_plugins::VehiclePlugin">
+        <ros>
+          <namespace>/$(arg namespace)</namespace>
+        </ros>
+        <vehicle_params>$(find qutms_sim)/config/vehicle_params.yaml</vehicle_params>
+        <update_rate>50.0</update_rate>
+        <steering_lock_time>1.5</steering_lock_time>
+      </plugin>
+    </gazebo>
+    <!-- Vehicle Control Plugin (requires vehicle dynamics plugin) -->
+    <gazebo>
+      <plugin filename="libgazebo_vehicle_control.so" name="gazebo_plugins::vehicle_plugins::VehicleControlPlugin">
+        <ros>
+          <namespace>/$(arg namespace)</namespace>
+        </ros>
+        <control_delay>0.035</control_delay>
+        <enable_ackermann>true</enable_ackermann>
+        <enable_twist>true</enable_twist>
+        <ackermann_topic>control/ackermann_cmd</ackermann_topic>
+        <twist_topic>control/twist_cmd</twist_topic>
+      </plugin>
+    </gazebo>
+  </xacro:if>
   <!-- INS Odometry Plugin -->
   <!--
@@ -136,7 +147,10 @@
     </plugin>
   </gazebo>
-  <!-- gz_ros2_control Gazebo Plugin -->
+  <!-- ============================================================= -->
+  <!-- ROS 2 CONTROL BACKEND (gz_ros2_control, physics-based)        -->
+  <!-- ============================================================= -->
   <!--
-    gz_ros2_control plugin - bridges ROS 2 Control with Gazebo simulation
+    gz_ros2_control plugin - bridges ROS 2 Control with Gazebo simulation.
+    Only active when control_mode == "ros2_control".
     Provides command and state interfaces for physics-based vehicle control:
     - Steering joints: position commands (target angle)
@@ -148,12 +162,14 @@
     - wheel effort controllers: Direct torque control for individual wheels
   -->
-  <gazebo>
-    <plugin filename="gz_ros2_control-system"
-            name="gz_ros2_control::GazeboSimROS2ControlPlugin">
-      <parameters>$(find qutms_sim)/config/ros2_controllers.yaml</parameters>
-      <ros>
-        <namespace>/$(arg namespace)</namespace>
-      </ros>
-    </plugin>
-  </gazebo>
+  <xacro:if value="${control_mode == 'ros2_control'}">
+    <gazebo>
+      <plugin filename="gz_ros2_control-system"
+              name="gz_ros2_control::GazeboSimROS2ControlPlugin">
+        <parameters>$(find qutms_sim)/config/ros2_controllers.yaml</parameters>
+        <ros>
+          <namespace>/$(arg namespace)</namespace>
+        </ros>
+      </plugin>
+    </gazebo>
+  </xacro:if>
 </robot>

File: qutms_sim/urdf/ros2_control.urdf.xacro (robot description, xacro)
@@ -19,4 +19,12 @@
   -->
   <xacro:arg name="namespace" default="sim"/>
+  <!--
+    Only declare the ros2_control hardware interfaces when the gz_ros2_control
+    backend is selected. In "dynamic_model" mode these joints are driven
+    kinematically and no controller_manager exists.
+  -->
+  <xacro:arg name="control_mode" default="dynamic_model"/>
+  <xacro:property name="control_mode" value="$(arg control_mode)"/>
+  <xacro:if value="${control_mode == 'ros2_control'}">
   <!-- ROS 2 Control System Definition -->
   <ros2_control name="GazeboSimSystem" type="system">
@@ -56,3 +64,4 @@
     </joint>
   </ros2_control>
+  </xacro:if>
 </robot>
