Commit message: WIP: Attempting to get ackermann control working. Effort control works with physics engine but ackermann uses velocity.

File: qutms_sim/urdf/components/wheels.urdf.xacro (robot description, xacro)
@@ -46,8 +46,4 @@
     <gazebo reference="${lr_prefix}_${fr_prefix}_wheel">
       <material>Gazebo/Black</material>
-      <mu1>${wheel_friction_mu1}</mu1>
-      <mu2>${wheel_friction_mu2}</mu2>
-      <!-- <minDepth>0.005</minDepth> -->
-      <kp>${wheel_friction_kp}</kp>
     </gazebo>
   </xacro:macro>
@@ -101,5 +97,6 @@
       <child link="${lr_prefix}_front_wheel"/>
       <axis xyz="0 1 0"/>
-      <limit lower="0" upper="0" effort="10000000" velocity="1000000"/>
+      <limit effort="200" velocity="100"/>
+      <dynamics damping="0.1" friction="0.0"/>
     </joint>
     <xacro:wheel lr_prefix="${lr_prefix}" fr_prefix="front"/>
@@ -116,5 +113,6 @@
       <child link="${lr_prefix}_rear_wheel"/>
       <axis xyz="0 1 0"/>
-      <limit lower="0" upper="0" effort="10000000" velocity="1000000"/>
+      <limit effort="200" velocity="100"/>
+      <dynamics damping="0.1" friction="0.0"/>
     </joint>
     <xacro:wheel lr_prefix="${lr_prefix}" fr_prefix="rear"/>

File: qutms_sim/urdf/robot.urdf.xacro (robot description, xacro)
@@ -63,5 +63,5 @@
     <inertial>
       <origin xyz="0 0 0" rpy="0 0 0" />
-      <mass value="200" />
+      <!-- <mass value="200" />
       <inertia
           ixx="16.3"
@@ -70,5 +70,13 @@
           iyy="33.6"
           iyz="0"
-          izz="47.9" />
+          izz="47.9" /> -->
+      <mass value="1" />
+      <inertia
+          ixx="1.3"
+          ixy="0"
+          ixz="0"
+          iyy="1.6"
+          iyz="0"
+          izz="1.9" />
     </inertial>
   </link>

File: qutms_sim/urdf/ros2_control.urdf.xacro (robot description, xacro)
@@ -41,13 +41,10 @@
       <state_interface name="velocity" />
     </joint>
-    <!-- Wheel joints - velocity + effort control for flexibility -->
+    <!-- Wheel joints - both velocity and effort (controller chooses based on config) -->
     <joint name="front_left_wheel_joint">
-      <command_interface name="velocity">
-        <param name="min">-50</param>  <!-- rad/s - adjust based on vehicle specs -->
-        <param name="max">50</param>
-      </command_interface>
+      <command_interface name="velocity" />
       <command_interface name="effort">
-        <param name="min">-100</param>  <!-- Nm - adjust based on vehicle specs -->
-        <param name="max">100</param>
+        <param name="min">-200</param>
+        <param name="max">200</param>
       </command_interface>
       <state_interface name="position" />
@@ -55,11 +52,8 @@
     </joint>
     <joint name="front_right_wheel_joint">
-      <command_interface name="velocity">
-        <param name="min">-50</param>
-        <param name="max">50</param>
-      </command_interface>
+      <command_interface name="velocity" />
       <command_interface name="effort">
-        <param name="min">-100</param>
-        <param name="max">100</param>
+        <param name="min">-200</param>
+        <param name="max">200</param>
       </command_interface>
       <state_interface name="position" />
@@ -67,11 +61,8 @@
     </joint>
     <joint name="rear_left_wheel_joint">
-      <command_interface name="velocity">
-        <param name="min">-50</param>
-        <param name="max">50</param>
-      </command_interface>
+      <command_interface name="velocity" />
       <command_interface name="effort">
-        <param name="min">-100</param>
-        <param name="max">100</param>
+        <param name="min">-200</param>
+        <param name="max">200</param>
       </command_interface>
       <state_interface name="position" />
@@ -79,11 +70,8 @@
     </joint>
     <joint name="rear_right_wheel_joint">
-      <command_interface name="velocity">
-        <param name="min">-50</param>
-        <param name="max">50</param>
-      </command_interface>
+      <command_interface name="velocity" />
       <command_interface name="effort">
-        <param name="min">-100</param>
-        <param name="max">100</param>
+        <param name="min">-200</param>
+        <param name="max">200</param>
       </command_interface>
       <state_interface name="position" />

Commit message: WIP: stripped back components. Vehicle wheel physics operates as expected

File: qutms_sim/urdf/components/wheels.urdf.xacro (robot description, xacro)
@@ -5,17 +5,14 @@
   <xacro:property name="chassis_width" value="1.6"/>
   <xacro:property name="wheelbase" value="1.580"/>
-  <xacro:property name="wheel_mass" value="10.0"/>
+  <xacro:property name="wheel_mass" value="3.0"/>
   <xacro:property name="wheel_diameter" value="0.4064"/>
   <xacro:property name="wheel_width" value="0.2"/>
-  <xacro:property name="wheel_friction_mu1" value="2"/>
-  <xacro:property name="wheel_friction_mu2" value="2"/>
-  <xacro:property name="wheel_friction_kp" value="1e8"/>
-  <xacro:property name="steering_hinge_mass" value="1"/>
+  <xacro:property name="wheel_friction_mu" value="2"/>
+  <xacro:property name="steering_mass" value="1"/>
   <material name="black">
       <color rgba="0 0 0 1"/>
   </material>
   <!-- Individual wheel constructor -->
-  <xacro:macro name="wheel"
-                params="lr_prefix fr_prefix">
+  <xacro:macro name="wheel" params="lr_prefix fr_prefix">
     <link name="${lr_prefix}_${fr_prefix}_wheel">
       <inertial>
@@ -42,4 +39,13 @@
           <cylinder radius="${wheel_diameter / 2}" length="${wheel_width}"/>
         </geometry>
+        <!-- GZ params -->
+        <surface>
+          <friction>
+            <ode>
+              <mu>${wheel_friction_mu}</mu>
+              <mu2>${wheel_friction_mu}</mu2>
+            </ode>
+          </friction>
+        </surface>
       </collision>
     </link>
@@ -52,11 +58,7 @@
   <!-- ********************************* -->
   <!-- Description of how a front wheel is connected to the chassis -->
-  <xacro:macro name="front_wheel"
-                params="lr_prefix lr_reflect">
+  <xacro:macro name="front_wheel" params="lr_prefix lr_reflect">
     <joint name="${lr_prefix}_steering_hinge_joint" type="revolute">
-      <origin xyz="${wheelbase / 2}
-                    ${lr_reflect * ((chassis_width - wheel_width) / 2)}
-                    0"
-              rpy="0 0 0"/>
+      <origin xyz="${wheelbase / 2} ${lr_reflect * ((chassis_width - wheel_width) / 2)} 0" rpy="0 0 0"/>
       <parent link="chassis"/>
       <child link="${lr_prefix}_steering_hinge"/>
@@ -65,54 +67,26 @@
     </joint>
     <link name="${lr_prefix}_steering_hinge">
-      <!-- Small visual/collision to ensure proper entity registration in GZ Sim -->
-      <visual>
-        <origin xyz="0 0 0" rpy="0 0 0"/>
-        <geometry>
-          <sphere radius="0.02"/>
-        </geometry>
-        <material name="black"/>
-      </visual>
-      <collision>
-        <origin xyz="0 0 0" rpy="0 0 0"/>
-        <geometry>
-          <sphere radius="0.02"/>
-        </geometry>
-      </collision>
       <inertial>
-        <origin xyz="0 0 0" rpy="0 0 0" />
-        <mass value="${steering_hinge_mass}"/>
-        <inertia
-            ixx="0.04"
-            ixy="0.0"
-            ixz="0.0"
-            iyy="0.04"
-            iyz="0.0"
-            izz="0.04"   />
+        <mass value="${steering_mass}"/>
+        <inertia ixx="0.001" ixy="0.0" ixz="0.0" iyy="0.001" iyz="0.0" izz="0.002" />
       </inertial>
     </link>
     <joint name="front_${lr_prefix}_wheel_joint" type="continuous">
-      <origin xyz="0 0 0"
-              rpy="0 0 0"/>
+      <origin xyz="0 0 0" rpy="-1.57 0 0"/>
       <parent link="${lr_prefix}_steering_hinge"/>
       <child link="${lr_prefix}_front_wheel"/>
-      <axis xyz="0 1 0"/>
-      <limit effort="200" velocity="100"/>
-      <dynamics damping="0.1" friction="0.0"/>
+      <axis xyz="0 0 1"/>
+      <dynamics damping="0.2"/>
     </joint>
     <xacro:wheel lr_prefix="${lr_prefix}" fr_prefix="front"/>
   </xacro:macro>
   <!-- Description of how a rear wheel is connected to the chassis -->
-  <xacro:macro name="rear_wheel"
-                params="lr_prefix lr_reflect">
+  <xacro:macro name="rear_wheel" params="lr_prefix lr_reflect">
     <joint name="rear_${lr_prefix}_wheel_joint" type="continuous">
-      <origin xyz="${-1 * wheelbase / 2}
-                    ${lr_reflect * ((chassis_width - wheel_width) / 2)}
-                    0"
-              rpy="0 0 0"/>
+      <origin xyz="${-1 * wheelbase / 2} ${lr_reflect * ((chassis_width - wheel_width) / 2)} 0" rpy="0 0 0"/>
       <parent link="chassis"/>
       <child link="${lr_prefix}_rear_wheel"/>
       <axis xyz="0 1 0"/>
-      <limit effort="200" velocity="100"/>
-      <dynamics damping="0.1" friction="0.0"/>
+      <dynamics damping="0.1"/>
     </joint>
     <xacro:wheel lr_prefix="${lr_prefix}" fr_prefix="rear"/>

File: qutms_sim/urdf/robot.urdf.xacro (robot description, xacro)
@@ -9,6 +9,6 @@
   <!-- Imports -->
   <xacro:include filename="$(find qutms_sim)/urdf/components/wheels.urdf.xacro"/>
-  <xacro:include filename="$(find qutms_sim)/urdf/components/lidar.urdf.xacro"/>
-  <xacro:include filename="$(find qutms_sim)/urdf/gz_plugins.urdf.xacro"/>
+  <!-- <xacro:include filename="$(find qutms_sim)/urdf/components/lidar.urdf.xacro"/> -->
+  <!-- <xacro:include filename="$(find qutms_sim)/urdf/gz_plugins.urdf.xacro"/> -->
   <xacro:include filename="$(find qutms_sim)/urdf/ros2_control.urdf.xacro"/>
   <!-- Vehicle Elements -->
@@ -24,6 +24,5 @@
     <child link="chassis"/>
     <!-- chassis link at wheel centre height above ground -->
-    <origin xyz="0 0 ${wheel_diameter/2}"
-            rpy="0 0 0"/>
+    <origin xyz="0 0 ${wheel_diameter/2}" rpy="0 0 0"/>
     <axis xyz="1 0 0"/>
   </joint>
@@ -63,5 +62,5 @@
     <inertial>
       <origin xyz="0 0 0" rpy="0 0 0" />
-      <!-- <mass value="200" />
+      <mass value="200" />
       <inertia
           ixx="16.3"
@@ -70,13 +69,5 @@
           iyy="33.6"
           iyz="0"
-          izz="47.9" /> -->
-      <mass value="1" />
-      <inertia
-          ixx="1.3"
-          ixy="0"
-          ixz="0"
-          iyy="1.6"
-          iyz="0"
-          izz="1.9" />
+          izz="47.9" />
     </inertial>
   </link>
@@ -87,6 +78,27 @@
   <xacro:rear_wheel lr_prefix="right" lr_reflect="-1" />
   <!-- LiDAR -->
-  <xacro:LiDAR parent="chassis" prefix="velodyne" namespace="$(arg namespace)">
+  <!-- <xacro:LiDAR parent="chassis" prefix="velodyne" namespace="$(arg namespace)">
     <origin xyz="1.590 0.0 0.0" rpy="0 0 0"/>
-  </xacro:LiDAR>
+  </xacro:LiDAR> -->
+  <!-- gz_ros2_control Gazebo Plugin -->
+  <gazebo>
+    <!--
+      gz_ros2_control plugin - bridges ROS 2 Control with Gazebo simulation
+      Provides command and state interfaces for physics-based vehicle control:
+      - Steering joints: position commands (target angle)
+      - Wheel joints: effort commands (torque for propulsion/braking)
+      - State feedback: position and velocity for all joints
+      Controllers (configured in ros2_controllers.yaml):
+      - joint_state_broadcaster: Publishes to /joint_states for robot_state_publisher
+      - ackermann_steering_controller: Bicycle model control via /cmd_vel
+      - wheel effort controllers: Direct torque control for individual wheels
+    -->
+    <plugin filename="gz_ros2_control-system"
+            name="gz_ros2_control::GazeboSimROS2ControlPlugin">
+      <parameters>$(find qutms_sim)/config/ros2_controllers.yaml</parameters>
+      <ros>
+        <namespace>/$(arg namespace)</namespace>
+      </ros>
+    </plugin>
+  </gazebo>
 </robot>

File: qutms_sim/urdf/ros2_control.urdf.xacro (robot description, xacro)
@@ -24,57 +24,34 @@
       <plugin>gz_ros2_control/GazeboSimSystem</plugin>
     </hardware>
-    <!-- Steering joints - position control for steering angle -->
+    <!-- Steering joints - position command (like demo) -->
     <joint name="left_steering_hinge_joint">
-      <command_interface name="position">
-        <param name="min">-0.6</param>  <!-- ~34 degrees -->
-        <param name="max">0.6</param>
-      </command_interface>
+      <command_interface name="position" />
       <state_interface name="position" />
       <state_interface name="velocity" />
     </joint>
     <joint name="right_steering_hinge_joint">
-      <command_interface name="position">
-        <param name="min">-0.6</param>
-        <param name="max">0.6</param>
-      </command_interface>
+      <command_interface name="position" />
       <state_interface name="position" />
       <state_interface name="velocity" />
     </joint>
-    <!-- Wheel joints - both velocity and effort (controller chooses based on config) -->
+    <!-- Front wheels - state feedback only (like demo) -->
     <joint name="front_left_wheel_joint">
-      <command_interface name="velocity" />
-      <command_interface name="effort">
-        <param name="min">-200</param>
-        <param name="max">200</param>
-      </command_interface>
       <state_interface name="position" />
       <state_interface name="velocity" />
     </joint>
     <joint name="front_right_wheel_joint">
-      <command_interface name="velocity" />
-      <command_interface name="effort">
-        <param name="min">-200</param>
-        <param name="max">200</param>
-      </command_interface>
       <state_interface name="position" />
       <state_interface name="velocity" />
     </joint>
+    <!-- Rear wheels - velocity command only (like demo) -->
     <joint name="rear_left_wheel_joint">
       <command_interface name="velocity" />
-      <command_interface name="effort">
-        <param name="min">-200</param>
-        <param name="max">200</param>
-      </command_interface>
+      <state_interface name="velocity" />
       <state_interface name="position" />
-      <state_interface name="velocity" />
     </joint>
     <joint name="rear_right_wheel_joint">
       <command_interface name="velocity" />
-      <command_interface name="effort">
-        <param name="min">-200</param>
-        <param name="max">200</param>
-      </command_interface>
+      <state_interface name="velocity" />
       <state_interface name="position" />
-      <state_interface name="velocity" />
     </joint>
   </ros2_control>

Commit message: Patch for Ackermann controller, now drives properly

File: qutms_sim/urdf/components/wheels.urdf.xacro (robot description, xacro)
@@ -73,8 +73,8 @@
     </link>
     <joint name="front_${lr_prefix}_wheel_joint" type="continuous">
-      <origin xyz="0 0 0" rpy="-1.57 0 0"/>
+      <origin xyz="0 0 0" rpy="0 0 0"/>
       <parent link="${lr_prefix}_steering_hinge"/>
       <child link="${lr_prefix}_front_wheel"/>
-      <axis xyz="0 0 1"/>
+      <axis xyz="0 1 0"/>
       <dynamics damping="0.2"/>
     </joint>

File: qutms_sim/urdf/gz_plugins.urdf.xacro (robot description, xacro)
@@ -51,12 +51,12 @@
   -->
   <!-- INS Odometry Plugin -->
+  <!--
+    Simulated INS sensor with configurable Gaussian noise.
+    Reads: Pose, LinearVelocity, AngularVelocity (ECM state components)
+    Publishes: /$(arg namespace)/odometry (nav_msgs/Odometry) - with noise
+                /$(arg namespace)/odometry/ground_truth (nav_msgs/Odometry) - perfect data
+    Noise model: Position, velocity, and orientation noise from vehicle_params.yaml
+  -->
   <gazebo>
-    <!--
-      Simulated INS sensor with configurable Gaussian noise.
-      Reads: Pose, LinearVelocity, AngularVelocity (ECM state components)
-      Publishes: /$(arg namespace)/odometry (nav_msgs/Odometry) - with noise
-                 /$(arg namespace)/odometry/ground_truth (nav_msgs/Odometry) - perfect data
-      Noise model: Position, velocity, and orientation noise from vehicle_params.yaml
-    -->
     <plugin filename="libgazebo_ins_odometry.so" name="gazebo_plugins::vehicle_plugins::INSOdometryPlugin">
       <ros>
@@ -73,11 +73,11 @@
   </gazebo>
   <!-- TF Broadcaster Plugin -->
+  <!--
+    Publishes vehicle transform tree.
+    Reads: Pose (ECM component)
+    Publishes: /tf (map → odom → base_footprint)
+    Note: Joint transforms handled by robot_state_publisher via gz_ros2_control
+  -->
   <gazebo>
-    <!--
-      Publishes vehicle transform tree.
-      Reads: Pose (ECM component)
-      Publishes: /tf (map → odom → base_footprint)
-      Note: Joint transforms handled by robot_state_publisher via gz_ros2_control
-    -->
     <plugin filename="libgazebo_tf_broadcaster.so" name="gazebo_plugins::vehicle_plugins::TFBroadcasterPlugin">
       <ros>
@@ -92,12 +92,12 @@
   </gazebo>
   <!-- Cone Detection Plugin -->
+  <!--
+    Simulates cone detection with configurable sensor characteristics.
+    Reads: Track model (cone positions), Vehicle pose
+    Publishes: /$(arg namespace)/track/ground_truth (driverless_msgs/ConeDetectionStamped)
+                /$(arg namespace)/detections/ground_truth (driverless_msgs/ConeDetectionStamped)
+    Features: FOV filtering, range filtering, bearing/range noise, color detection toggle
+  -->
   <gazebo>
-    <!--
-      Simulates cone detection with configurable sensor characteristics.
-      Reads: Track model (cone positions), Vehicle pose
-      Publishes: /$(arg namespace)/track/ground_truth (driverless_msgs/ConeDetectionStamped)
-                 /$(arg namespace)/detections/ground_truth (driverless_msgs/ConeDetectionStamped)
-      Features: FOV filtering, range filtering, bearing/range noise, color detection toggle
-    -->
     <plugin filename="libgazebo_cone_detection.so" name="gazebo_plugins::vehicle_plugins::ConeDetectionPlugin">
       <ros>
@@ -119,14 +119,14 @@
   </gazebo>
   <!-- Simulation Reset Plugin -->
+  <!--
+    Centralized simulation reset for vehicle and track.
+    Service: /$(arg namespace)/reset_simulation (std_srvs/Trigger)
+    Resets:
+    - VehicleState ECM component to initial values
+    - WorldPoseCmd/WorldLinearVelocityCmd/WorldAngularVelocityCmd to spawn position
+    - All cone link poses to original track layout
+    Enables quick simulation restart without relaunching
+  -->
   <gazebo>
-    <!--
-      Centralized simulation reset for vehicle and track.
-      Service: /$(arg namespace)/reset_simulation (std_srvs/Trigger)
-      Resets:
-      - VehicleState ECM component to initial values
-      - WorldPoseCmd/WorldLinearVelocityCmd/WorldAngularVelocityCmd to spawn position
-      - All cone link poses to original track layout
-      Enables quick simulation restart without relaunching
-    -->
     <plugin filename="libgazebo_sim_reset.so" name="gazebo_plugins::vehicle_plugins::SimResetPlugin">
       <ros>
@@ -137,16 +137,16 @@
   </gazebo>
   <!-- gz_ros2_control Gazebo Plugin -->
+  <!--
+    gz_ros2_control plugin - bridges ROS 2 Control with Gazebo simulation
+    Provides command and state interfaces for physics-based vehicle control:
+    - Steering joints: position commands (target angle)
+    - Wheel joints: effort commands (torque for propulsion/braking)
+    - State feedback: position and velocity for all joints
+    Controllers (configured in ros2_controllers.yaml):
+    - joint_state_broadcaster: Publishes to /joint_states for robot_state_publisher
+    - ackermann_steering_controller: Bicycle model control via /cmd_vel
+    - wheel effort controllers: Direct torque control for individual wheels
+  -->
   <gazebo>
-    <!--
-      gz_ros2_control plugin - bridges ROS 2 Control with Gazebo simulation
-      Provides command and state interfaces for physics-based vehicle control:
-      - Steering joints: position commands (target angle)
-      - Wheel joints: effort commands (torque for propulsion/braking)
-      - State feedback: position and velocity for all joints
-      Controllers (configured in ros2_controllers.yaml):
-      - joint_state_broadcaster: Publishes to /joint_states for robot_state_publisher
-      - ackermann_steering_controller: Bicycle model control via /cmd_vel
-      - wheel effort controllers: Direct torque control for individual wheels
-    -->
     <plugin filename="gz_ros2_control-system"
             name="gz_ros2_control::GazeboSimROS2ControlPlugin">

File: qutms_sim/urdf/robot.urdf.xacro (robot description, xacro)
@@ -9,6 +9,6 @@
   <!-- Imports -->
   <xacro:include filename="$(find qutms_sim)/urdf/components/wheels.urdf.xacro"/>
-  <!-- <xacro:include filename="$(find qutms_sim)/urdf/components/lidar.urdf.xacro"/> -->
-  <!-- <xacro:include filename="$(find qutms_sim)/urdf/gz_plugins.urdf.xacro"/> -->
+  <xacro:include filename="$(find qutms_sim)/urdf/components/lidar.urdf.xacro"/>
+  <xacro:include filename="$(find qutms_sim)/urdf/gz_plugins.urdf.xacro"/>
   <xacro:include filename="$(find qutms_sim)/urdf/ros2_control.urdf.xacro"/>
   <!-- Vehicle Elements -->
@@ -78,27 +78,6 @@
   <xacro:rear_wheel lr_prefix="right" lr_reflect="-1" />
   <!-- LiDAR -->
-  <!-- <xacro:LiDAR parent="chassis" prefix="velodyne" namespace="$(arg namespace)">
+  <xacro:LiDAR parent="chassis" prefix="velodyne" namespace="$(arg namespace)">
     <origin xyz="1.590 0.0 0.0" rpy="0 0 0"/>
-  </xacro:LiDAR> -->
-  <!-- gz_ros2_control Gazebo Plugin -->
-  <gazebo>
-    <!--
-      gz_ros2_control plugin - bridges ROS 2 Control with Gazebo simulation
-      Provides command and state interfaces for physics-based vehicle control:
-      - Steering joints: position commands (target angle)
-      - Wheel joints: effort commands (torque for propulsion/braking)
-      - State feedback: position and velocity for all joints
-      Controllers (configured in ros2_controllers.yaml):
-      - joint_state_broadcaster: Publishes to /joint_states for robot_state_publisher
-      - ackermann_steering_controller: Bicycle model control via /cmd_vel
-      - wheel effort controllers: Direct torque control for individual wheels
-    -->
-    <plugin filename="gz_ros2_control-system"
-            name="gz_ros2_control::GazeboSimROS2ControlPlugin">
-      <parameters>$(find qutms_sim)/config/ros2_controllers.yaml</parameters>
-      <ros>
-        <namespace>/$(arg namespace)</namespace>
-      </ros>
-    </plugin>
-  </gazebo>
+  </xacro:LiDAR>
 </robot>
